File: electronics/kicad/wollemi_eps_card.kicad_pcb (KiCad board)
At the start: 4 copper layers, 100 x 100 mm, 12 parts, among them J1 WL-P, U1 MPPT_BUCK, U2 MPPT_BUCK, U3 MPPT_BUCK, U4 CHG_BAL, U5 IDEAL_DIODE, U6 EFUSE_OVPUVP, U7 TELEM_MCU

Commit message: EPS card candidate part selection (v0): LT8490 MPPT/charger, BQ29209-Q1 2S balancer, LTC4359 ideal diode, TPS2597x eFuse, STM32G0B1 telemetry MCU, discrete AND-gated burn-wire driver; pinned pack C to 2S1P for parts commonality; floor plan labels updated to match, still DRC clean
Parts:
- U1, U2, U3: value MPPT_BUCK -> LT8490; footprint Wollemi:MPPT_BUCK_placeholder -> Wollemi:LT8490_placeholder
- U4: value CHG_BAL -> BQ29209-Q1; footprint Wollemi:CHG_BAL_placeholder -> Wollemi:BQ29209-Q1_placeholder
- U5: value IDEAL_DIODE -> LTC4359; footprint Wollemi:IDEAL_DIODE_placeholder -> Wollemi:LTC4359_placeholder
- U6: value EFUSE_OVPUVP -> TPS2597x; footprint Wollemi:EFUSE_OVPUVP_placeholder -> Wollemi:TPS2597x_placeholder
- U7: value TELEM_MCU -> STM32G0B1; footprint Wollemi:TELEM_MCU_placeholder -> Wollemi:STM32G0B1_placeholder
Changed lines of the file:
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@@
     (pad "60" smd rect (at 1.500 18.415) (size 1.4 0.5) (layers "F.Cu" "F.Mask" "F.Paste") (net 31 "RSV"))
   )
-  (footprint "Wollemi:MPPT_BUCK_placeholder" (layer "F.Cu") (at 40 22)
+  (footprint "Wollemi:LT8490_placeholder" (layer "F.Cu") (at 40 22)
     (property "Reference" "U1" (at 0 -10.60 0) (layer "F.SilkS") (effects (font (size 1 1) (thickness 0.15))))
-    (property "Value" "MPPT_BUCK" (at 0 10.60 0) (layer "F.Fab") (effects (font (size 0.9 0.9) (thickness 0.13))))
+    (property "Value" "LT8490" (at 0 10.60 0) (layer "F.Fab") (effects (font (size 0.9 0.9) (thickness 0.13))))
     (attr exclude_from_pos_files exclude_from_bom)
     (fp_rect (start -13.00 -9.00) (end 13.00 9.00) (stroke (width 0.15) (type default)) (fill no) (layer "F.SilkS"))
     (fp_rect (start -13.00 -9.00) (end 13.00 9.00) (stroke (width 0.05) (type default)) (fill no) (layer "F.CrtYd"))
-    (fp_text user "MPPT ch1: 8-40V->6.4V, ~24W" (at 0 0 0) (layer "F.Fab") (effects (font (size 0.9 0.9) (thickness 0.15))))
+    (fp_text user "MPPT ch1: 8-40V->6.4V, ~24W (cand. LT8490)" (at 0 0 0) (layer "F.Fab") (effects (font (size 0.9 0.9) (thickness 0.15))))
   )
-  (footprint "Wollemi:MPPT_BUCK_placeholder" (layer "F.Cu") (at 40 46)
+  (footprint "Wollemi:LT8490_placeholder" (layer "F.Cu") (at 40 46)
     (property "Reference" "U2" (at 0 -10.60 0) (layer "F.SilkS") (effects (font (size 1 1) (thickness 0.15))))
-    (property "Value" "MPPT_BUCK" (at 0 10.60 0) (layer "F.Fab") (effects (font (size 0.9 0.9) (thickness 0.13))))
+    (property "Value" "LT8490" (at 0 10.60 0) (layer "F.Fab") (effects (font (size 0.9 0.9) (thickness 0.13))))
     (attr exclude_from_pos_files exclude_from_bom)
     (fp_rect (start -13.00 -9.00) (end 13.00 9.00) (stroke (width 0.15) (type default)) (fill no) (layer "F.SilkS"))
     (fp_rect (start -13.00 -9.00) (end 13.00 9.00) (stroke (width 0.05) (type default)) (fill no) (layer "F.CrtYd"))
-    (fp_text user "MPPT ch2: 8-40V->6.4V, ~24W" (at 0 0 0) (layer "F.Fab") (effects (font (size 0.9 0.9) (thickness 0.15))))
+    (fp_text user "MPPT ch2: 8-40V->6.4V, ~24W (cand. LT8490)" (at 0 0 0) (layer "F.Fab") (effects (font (size 0.9 0.9) (thickness 0.15))))
   )
-  (footprint "Wollemi:MPPT_BUCK_placeholder" (layer "F.Cu") (at 40 70)
+  (footprint "Wollemi:LT8490_placeholder" (layer "F.Cu") (at 40 70)
     (property "Reference" "U3" (at 0 -10.60 0) (layer "F.SilkS") (effects (font (size 1 1) (thickness 0.15))))
-    (property "Value" "MPPT_BUCK" (at 0 10.60 0) (layer "F.Fab") (effects (font (size 0.9 0.9) (thickness 0.13))))
+    (property "Value" "LT8490" (at 0 10.60 0) (layer "F.Fab") (effects (font (size 0.9 0.9) (thickness 0.13))))
     (attr exclude_from_pos_files exclude_from_bom)
     (fp_rect (start -13.00 -9.00) (end 13.00 9.00) (stroke (width 0.15) (type default)) (fill no) (layer "F.SilkS"))
     (fp_rect (start -13.00 -9.00) (end 13.00 9.00) (stroke (width 0.05) (type default)) (fill no) (layer "F.CrtYd"))
-    (fp_text user "MPPT ch3: 8-40V->6.4V, ~24W" (at 0 0 0) (layer "F.Fab") (effects (font (size 0.9 0.9) (thickness 0.15))))
+    (fp_text user "MPPT ch3: 8-40V->6.4V, ~24W (cand. LT8490)" (at 0 0 0) (layer "F.Fab") (effects (font (size 0.9 0.9) (thickness 0.15))))
   )
-  (footprint "Wollemi:CHG_BAL_placeholder" (layer "F.Cu") (at 68 22)
+  (footprint "Wollemi:BQ29209-Q1_placeholder" (layer "F.Cu") (at 68 22)
     (property "Reference" "U4" (at 0 -11.60 0) (layer "F.SilkS") (effects (font (size 1 1) (thickness 0.15))))
-    (property "Value" "CHG_BAL" (at 0 11.60 0) (layer "F.Fab") (effects (font (size 0.9 0.9) (thickness 0.13))))
+    (property "Value" "BQ29209-Q1" (at 0 11.60 0) (layer "F.Fab") (effects (font (size 0.9 0.9) (thickness 0.13))))
     (attr exclude_from_pos_files exclude_from_bom)
     (fp_rect (start -14.00 -10.00) (end 14.00 10.00) (stroke (width 0.15) (type default)) (fill no) (layer "F.SilkS"))
     (fp_rect (start -14.00 -10.00) (end 14.00 10.00) (stroke (width 0.05) (type default)) (fill no) (layer "F.CrtYd"))
-    (fp_text user "Pack charger + balancer: CC-CV 7.3V, 3.3A" (at 0 0 0) (layer "F.Fab") (effects (font (size 0.9 0.9) (thickness 0.15))))
+    (fp_text user "2S balance corrector (cand. BQ29209-Q1)" (at 0 0 0) (layer "F.Fab") (effects (font (size 0.9 0.9) (thickness 0.15))))
   )
-  (footprint "Wollemi:IDEAL_DIODE_placeholder" (layer "F.Cu") (at 68 48)
+  (footprint "Wollemi:LTC4359_placeholder" (layer "F.Cu") (at 68 48)
     (property "Reference" "U5" (at 0 -8.60 0) (layer "F.SilkS") (effects (font (size 1 1) (thickness 0.15))))
-    (property "Value" "IDEAL_DIODE" (at 0 8.60 0) (layer "F.Fab") (effects (font (size 0.9 0.9) (thickness 0.13))))
+    (property "Value" "LTC4359" (at 0 8.60 0) (layer "F.Fab") (effects (font (size 0.9 0.9) (thickness 0.13))))
     (attr exclude_from_pos_files exclude_from_bom)
     (fp_rect (start -10.00 -7.00) (end 10.00 7.00) (stroke (width 0.15) (type default)) (fill no) (layer "F.SilkS"))
     (fp_rect (start -10.00 -7.00) (end 10.00 7.00) (stroke (width 0.05) (type default)) (fill no) (layer "F.CrtYd"))
-    (fp_text user "Ideal diode OR-ing to bus" (at 0 0 0) (layer "F.Fab") (effects (font (size 0.9 0.9) (thickness 0.15))))
+    (fp_text user "Ideal diode OR-ing (cand. LTC4359)" (at 0 0 0) (layer "F.Fab") (effects (font (size 0.9 0.9) (thickness 0.15))))
   )
-  (footprint "Wollemi:EFUSE_OVPUVP_placeholder" (layer "F.Cu") (at 68 66)
+  (footprint "Wollemi:TPS2597x_placeholder" (layer "F.Cu") (at 68 66)
     (property "Reference" "U6" (at 0 -9.60 0) (layer "F.SilkS") (effects (font (size 1 1) (thickness 0.15))))
-    (property "Value" "EFUSE_OVPUVP" (at 0 9.60 0) (layer "F.Fab") (effects (font (size 0.9 0.9) (thickness 0.13))))
+    (property "Value" "TPS2597x" (at 0 9.60 0) (layer "F.Fab") (effects (font (size 0.9 0.9) (thickness 0.13))))
     (attr exclude_from_pos_files exclude_from_bom)
     (fp_rect (start -12.00 -8.00) (end 12.00 8.00) (stroke (width 0.15) (type default)) (fill no) (layer "F.SilkS"))
     (fp_rect (start -12.00 -8.00) (end 12.00 8.00) (stroke (width 0.05) (type default)) (fill no) (layer "F.CrtYd"))
-    (fp_text user "eFuse + OVP/UVP, hardware only" (at 0 0 0) (layer "F.Fab") (effects (font (size 0.9 0.9) (thickness 0.15))))
+    (fp_text user "eFuse+OVP/UVP, HW only (cand. TPS2597x)" (at 0 0 0) (layer "F.Fab") (effects (font (size 0.9 0.9) (thickness 0.15))))
   )
-  (footprint "Wollemi:TELEM_MCU_placeholder" (layer "F.Cu") (at 40 92)
+  (footprint "Wollemi:STM32G0B1_placeholder" (layer "F.Cu") (at 40 92)
     (property "Reference" "U7" (at 0 -8.60 0) (layer "F.SilkS") (effects (font (size 1 1) (thickness 0.15))))
-    (property "Value" "TELEM_MCU" (at 0 8.60 0) (layer "F.Fab") (effects (font (size 0.9 0.9) (thickness 0.13))))
+    (property "Value" "STM32G0B1" (at 0 8.60 0) (layer "F.Fab") (effects (font (size 0.9 0.9) (thickness 0.13))))
     (attr exclude_from_pos_files exclude_from_bom)
     (fp_rect (start -11.00 -7.00) (end 11.00 7.00) (stroke (width 0.15) (type default)) (fill no) (layer "F.SilkS"))
     (fp_rect (start -11.00 -7.00) (end 11.00 7.00) (stroke (width 0.05) (type default)) (fill no) (layer "F.CrtYd"))
-    (fp_text user "Telemetry MCU: V/I/T, CAN-FD" (at 0 0 0) (layer "F.Fab") (effects (font (size 0.9 0.9) (thickness 0.15))))
+    (fp_text user "Telemetry MCU: V/I/T, CAN-FD (cand. STM32G0B1)" (at 0 0 0) (layer "F.Fab") (effects (font (size 0.9 0.9) (thickness 0.15))))
   )
 )
