File: electronics/kicad/wollemi_survival_card.kicad_pcb (KiCad board)
At the start: 4 copper layers, 100 x 100 mm, 11 parts, among them J1 WL-P, U1 CHG_C, U2 DIRECT_PATH, U3 IDEAL_DIODE, U4 BURNWIRE1, U5 BURNWIRE2, U6 TELEM_MCU

Commit message: EPS card candidate part selection (v0): LT8490 MPPT/charger, BQ29209-Q1 2S balancer, LTC4359 ideal diode, TPS2597x eFuse, STM32G0B1 telemetry MCU, discrete AND-gated burn-wire driver; pinned pack C to 2S1P for parts commonality; floor plan labels updated to match, still DRC clean
Parts:
- U1: value CHG_C -> LT8490; footprint Wollemi:CHG_C_placeholder -> Wollemi:LT8490_placeholder
- U2: value DIRECT_PATH -> LTC4359; footprint Wollemi:DIRECT_PATH_placeholder -> Wollemi:LTC4359_placeholder
- U3: value IDEAL_DIODE -> LTC4359; footprint Wollemi:IDEAL_DIODE_placeholder -> Wollemi:LTC4359_placeholder
- U4: value BURNWIRE1 -> MOSFET+AND; footprint Wollemi:BURNWIRE1_placeholder -> Wollemi:MOSFET+AND_placeholder
- U5: value BURNWIRE2 -> MOSFET+AND; footprint Wollemi:BURNWIRE2_placeholder -> Wollemi:MOSFET+AND_placeholder
- U6: value TELEM_MCU -> MSP430FR?; footprint Wollemi:TELEM_MCU_placeholder -> Wollemi:MSP430FR?_placeholder
Changed lines of the file:
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@@
     (pad "60" smd rect (at 1.500 18.415) (size 1.4 0.5) (layers "F.Cu" "F.Mask" "F.Paste") (net 31 "RSV"))
   )
-  (footprint "Wollemi:CHG_C_placeholder" (layer "F.Cu") (at 45 22)
+  (footprint "Wollemi:LT8490_placeholder" (layer "F.Cu") (at 45 22)
     (property "Reference" "U1" (at 0 -10.60 0) (layer "F.SilkS") (effects (font (size 1 1) (thickness 0.15))))
-    (property "Value" "CHG_C" (at 0 10.60 0) (layer "F.Fab") (effects (font (size 0.9 0.9) (thickness 0.13))))
+    (property "Value" "LT8490" (at 0 10.60 0) (layer "F.Fab") (effects (font (size 0.9 0.9) (thickness 0.13))))
     (attr exclude_from_pos_files exclude_from_bom)
     (fp_rect (start -13.00 -9.00) (end 13.00 9.00) (stroke (width 0.15) (type default)) (fill no) (layer "F.SilkS"))
     (fp_rect (start -13.00 -9.00) (end 13.00 9.00) (stroke (width 0.05) (type default)) (fill no) (layer "F.CrtYd"))
-    (fp_text user "Pack C charger: 4s2p ~9.6V, 1A" (at 0 0 0) (layer "F.Fab") (effects (font (size 0.9 0.9) (thickness 0.15))))
+    (fp_text user "Pack C charger 2S1P ~6.4V, 1A (cand. LT8490)" (at 0 0 0) (layer "F.Fab") (effects (font (size 0.9 0.9) (thickness 0.15))))
   )
-  (footprint "Wollemi:DIRECT_PATH_placeholder" (layer "F.Cu") (at 45 46)
+  (footprint "Wollemi:LTC4359_placeholder" (layer "F.Cu") (at 45 46)
     (property "Reference" "U2" (at 0 -9.60 0) (layer "F.SilkS") (effects (font (size 1 1) (thickness 0.15))))
-    (property "Value" "DIRECT_PATH" (at 0 9.60 0) (layer "F.Fab") (effects (font (size 0.9 0.9) (thickness 0.13))))
+    (property "Value" "LTC4359" (at 0 9.60 0) (layer "F.Fab") (effects (font (size 0.9 0.9) (thickness 0.13))))
     (attr exclude_from_pos_files exclude_from_bom)
     (fp_rect (start -11.00 -8.00) (end 11.00 8.00) (stroke (width 0.15) (type default)) (fill no) (layer "F.SilkS"))
     (fp_rect (start -11.00 -8.00) (end 11.00 8.00) (stroke (width 0.05) (type default)) (fill no) (layer "F.CrtYd"))
-    (fp_text user "Direct string path -> supervisor (sun-only)" (at 0 0 0) (layer "F.Fab") (effects (font (size 0.9 0.9) (thickness 0.15))))
+    (fp_text user "Direct path -> supervisor (cand. LTC4359)" (at 0 0 0) (layer "F.Fab") (effects (font (size 0.9 0.9) (thickness 0.15))))
   )
-  (footprint "Wollemi:IDEAL_DIODE_placeholder" (layer "F.Cu") (at 75 22)
+  (footprint "Wollemi:LTC4359_placeholder" (layer "F.Cu") (at 75 22)
     (property "Reference" "U3" (at 0 -8.60 0) (layer "F.SilkS") (effects (font (size 1 1) (thickness 0.15))))
-    (property "Value" "IDEAL_DIODE" (at 0 8.60 0) (layer "F.Fab") (effects (font (size 0.9 0.9) (thickness 0.13))))
+    (property "Value" "LTC4359" (at 0 8.60 0) (layer "F.Fab") (effects (font (size 0.9 0.9) (thickness 0.13))))
     (attr exclude_from_pos_files exclude_from_bom)
     (fp_rect (start -9.00 -7.00) (end 9.00 7.00) (stroke (width 0.15) (type default)) (fill no) (layer "F.SilkS"))
     (fp_rect (start -9.00 -7.00) (end 9.00 7.00) (stroke (width 0.05) (type default)) (fill no) (layer "F.CrtYd"))
-    (fp_text user "Ideal diode" (at 0 0 0) (layer "F.Fab") (effects (font (size 0.9 0.9) (thickness 0.15))))
+    (fp_text user "Ideal diode (cand. LTC4359)" (at 0 0 0) (layer "F.Fab") (effects (font (size 0.9 0.9) (thickness 0.15))))
   )
-  (footprint "Wollemi:BURNWIRE1_placeholder" (layer "F.Cu") (at 45 68)
+  (footprint "Wollemi:MOSFET+AND_placeholder" (layer "F.Cu") (at 45 68)
     (property "Reference" "U4" (at 0 -9.60 0) (layer "F.SilkS") (effects (font (size 1 1) (thickness 0.15))))
-    (property "Value" "BURNWIRE1" (at 0 9.60 0) (layer "F.Fab") (effects (font (size 0.9 0.9) (thickness 0.13))))
+    (property "Value" "MOSFET+AND" (at 0 9.60 0) (layer "F.Fab") (effects (font (size 0.9 0.9) (thickness 0.13))))
     (attr exclude_from_pos_files exclude_from_bom)
     (fp_rect (start -12.00 -8.00) (end 12.00 8.00) (stroke (width 0.15) (type default)) (fill no) (layer "F.SilkS"))
     (fp_rect (start -12.00 -8.00) (end 12.00 8.00) (stroke (width 0.05) (type default)) (fill no) (layer "F.CrtYd"))
-    (fp_text user "Burn-wire driver 1: 3 inhibits (timer, supervisor, sep-sw)" (at 0 0 0) (layer "F.Fab") (effects (font (size 0.9 0.9) (thickness 0.15))))
+    (fp_text user "Burn-wire 1: 3-input AND gate + FET (discrete)" (at 0 0 0) (layer "F.Fab") (effects (font (size 0.9 0.9) (thickness 0.15))))
   )
-  (footprint "Wollemi:BURNWIRE2_placeholder" (layer "F.Cu") (at 45 90)
+  (footprint "Wollemi:MOSFET+AND_placeholder" (layer "F.Cu") (at 45 90)
     (property "Reference" "U5" (at 0 -9.60 0) (layer "F.SilkS") (effects (font (size 1 1) (thickness 0.15))))
-    (property "Value" "BURNWIRE2" (at 0 9.60 0) (layer "F.Fab") (effects (font (size 0.9 0.9) (thickness 0.13))))
+    (property "Value" "MOSFET+AND" (at 0 9.60 0) (layer "F.Fab") (effects (font (size 0.9 0.9) (thickness 0.13))))
     (attr exclude_from_pos_files exclude_from_bom)
     (fp_rect (start -12.00 -8.00) (end 12.00 8.00) (stroke (width 0.15) (type default)) (fill no) (layer "F.SilkS"))
     (fp_rect (start -12.00 -8.00) (end 12.00 8.00) (stroke (width 0.05) (type default)) (fill no) (layer "F.CrtYd"))
-    (fp_text user "Burn-wire driver 2: 3 inhibits (same)" (at 0 0 0) (layer "F.Fab") (effects (font (size 0.9 0.9) (thickness 0.15))))
+    (fp_text user "Burn-wire 2: 3-input AND gate + FET (discrete)" (at 0 0 0) (layer "F.Fab") (effects (font (size 0.9 0.9) (thickness 0.15))))
   )
-  (footprint "Wollemi:TELEM_MCU_placeholder" (layer "F.Cu") (at 78 46)
+  (footprint "Wollemi:MSP430FR?_placeholder" (layer "F.Cu") (at 78 46)
     (property "Reference" "U6" (at 0 -8.60 0) (layer "F.SilkS") (effects (font (size 1 1) (thickness 0.15))))
-    (property "Value" "TELEM_MCU" (at 0 8.60 0) (layer "F.Fab") (effects (font (size 0.9 0.9) (thickness 0.13))))
+    (property "Value" "MSP430FR?" (at 0 8.60 0) (layer "F.Fab") (effects (font (size 0.9 0.9) (thickness 0.13))))
     (attr exclude_from_pos_files exclude_from_bom)
     (fp_rect (start -10.00 -7.00) (end 10.00 7.00) (stroke (width 0.15) (type default)) (fill no) (layer "F.SilkS"))
     (fp_rect (start -10.00 -7.00) (end 10.00 7.00) (stroke (width 0.05) (type default)) (fill no) (layer "F.CrtYd"))
-    (fp_text user "Telemetry MCU" (at 0 0 0) (layer "F.Fab") (effects (font (size 0.9 0.9) (thickness 0.15))))
+    (fp_text user "Telemetry: reuse supervisor? (open, see docs/eps-card.md)" (at 0 0 0) (layer "F.Fab") (effects (font (size 0.9 0.9) (thickness 0.15))))
   )
 )
